File: mix/mix.kicad_pcb (KiCad board)
At the start: 2 copper layers, 203 x 119.7 mm, 67 parts, among them SW1 RotaryEncoder_Switch_MP, SW10 RotaryEncoder_Switch_MP, SW11 SW_Push, SW12 SW_Push, SW13 RotaryEncoder_Switch_MP, SW14 SW_Push, SW15 SW_Push, SW16 RotaryEncoder_Switch_MP, SW17 SW_Push, SW18 SW_Push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

Commit message: images
Parts:
- removed VR1, VR2, VR3, VR4, VR5, VR6, VR7, VR8: RS45111A900F, KiCad:RS45111A900F
- added R1: ~, SlidePOT:RES-ADJ_PTA4543-2015CPB102, F.Cu at (84.5, 125.0)
- added R2: ~, SlidePOT:RES-ADJ_PTA4543-2015CPB102, F.Cu at (103.6, 125.0)
- added R3: ~, SlidePOT:RES-ADJ_PTA4543-2015CPB102, F.Cu at (122.6, 125.0)
- added R4: ~, SlidePOT:RES-ADJ_PTA4543-2015CPB102, F.Cu at (141.7, 125.0)
- added R5: ~, SlidePOT:RES-ADJ_PTA4543-2015CPB102, F.Cu at (160.7, 125.0)
- added R6: ~, SlidePOT:RES-ADJ_PTA4543-2015CPB102, F.Cu at (179.8, 125.0)
- added R7: ~, SlidePOT:RES-ADJ_PTA4543-2015CPB102, F.Cu at (198.8, 125.0)
- added R8: ~, SlidePOT:RES-ADJ_PTA4543-2015CPB102, F.Cu at (217.9, 125.0)
- moved D1 4.21 mm to (76.8, 103.6)
- moved D11 4.21 mm to (172.0, 103.6)
- moved D13 4.21 mm to (191.1, 103.6)
- moved D15 4.21 mm to (210.1, 103.6)
- moved D3 4.21 mm to (95.8, 103.6)
- moved D5 4.21 mm to (114.9, 103.6)
- moved D7 4.21 mm to (133.9, 103.6)
- moved D9 4.21 mm to (153.0, 103.6)
- moved D16 1.33 mm to (225.6, 98.2)
- moved D10 0.84 mm to (168.5, 98.8)
- moved D12 0.84 mm to (187.5, 98.8)
- moved D14 0.84 mm to (206.6, 98.8)
- moved D2 0.84 mm to (92.3, 98.8)
- moved D4 0.84 mm to (111.3, 98.8)
- moved D6 0.84 mm to (130.4, 98.8)
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Routing:
- net Net-(D8-DOUT): track 7.44 -> 2.25 mm
- net Net-(D14-DOUT): track 7.44 -> 2.25 mm
- net Net-(D10-DOUT): track 7.44 -> 2.25 mm
- net Net-(D2-DOUT): track 7.44 -> 2.25 mm
- net Net-(D4-DOUT): track 7.37 -> 2.25 mm
- net Net-(D6-DOUT): track 7.37 -> 2.25 mm
- net Net-(D12-DOUT): track 7.37 -> 2.25 mm
- net CH7F: track 145.5 -> 150.2 mm
- net CH6F: track 126.0 -> 130.6 mm
- net CH5F: track 106.4 -> 111.0 mm
- net CH4F: track 86.8 -> 91.5 mm
- net CH3F: track 67.2 -> 71.9 mm
- net CH2F: track 47.7 -> 52.3 mm
- net CH1F: track 28.1 -> 32.7 mm
- net CH0F: track 10.2 -> 14.2 mm
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