File: mix/mix.kicad_sch (KiCad schematic)
At the start: 67 parts, among them SW1 RotaryEncoder_Switch_MP, SW10 RotaryEncoder_Switch_MP, SW11 SW_Push, SW12 SW_Push, SW13 RotaryEncoder_Switch_MP, SW14 SW_Push, SW15 SW_Push, SW16 RotaryEncoder_Switch_MP, SW17 SW_Push, SW18 SW_Push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

Commit message: images
Parts:
- removed VR1, VR2, VR3, VR4, VR5, VR6, VR7, VR8: RS45111A900F, KiCad:RS45111A900F, symbol RS45111A900F:RS45111A900F
- added R1, R2, R3, R4, R5, R6, R7, R8: ~, SlidePOT:RES-ADJ_PTA4543-2015CPB102, symbol SlidePOT:PTA4543-2015DPB103
Connections:
- net +3V3: now also R1.3, R2.3, R3.3, R4.3, R5.3, R6.3, R7.3, R8.3
- net CH0F: now also R1.2
- net CH1F: now also R2.2
- net CH2F: now also R3.2
- net CH3F: now also R4.2
- net CH4F: now also R5.2
- net CH5F: now also R6.2
- net CH6F: now also R7.2
- net CH7F: now also R8.2
- net GND: now also R1.1, R2.1, R3.1, R4.1, R5.1, R6.1, R7.1, R8.1
- no-connect marks 27 -> 43
